File: Transmitter/KiCAD/Button Transmitter/button_transmitter.kicad_pcb (KiCad board)
At the start: 2 copper layers, 59.6 x 55.9 mm, 43 parts, among them J10 2.54mm, J2 1.27mm Pogo Pads, J3 2.54mm, J5 2.54mm, J7 SMA, J8 SMA, J9 SMA, SW1 SW_SPDT, U1 ATtiny212-SS, U2 Si5351B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

Commit message: Added JLC order number to gerber files
Other:
- board text added: "JLCJLCJLCJLC"
