File: Transmitter/KiCAD/Button Transmitter/Si5351B-ATtiny412 Dev Board/CR2032 Battery/button_transmitter.kicad_pcb (KiCad board)
At the start: 2 copper layers, 40 x 40 mm, 37 parts, among them J1 1.27mm Pogo Pads, J2 Conn_Coaxial, Q1 MMUN2238LT1G, U1 ATtiny412-SS, U2 Si5351B-B-GM1, U3 TLV62568DRL, Y1 25MHz

Commit message: Pause point in CR2032 layout
Parts:
- BT1: value JST Battery Connector -> CR2032; footprint Library:JST_PH_HORIZONTAL_WITH_BATTERY_3 -> Battery:BatteryHolder_Keystone_3034_1x20mm; moved to B.Cu
- J2: footprint Library:MountingHole_4.3mm_Pad_Coaxial_2 -> Library:RF_Solder_Pad
- U4: footprint Library:Case -> Library:Case_CR2032
- moved J2 49.8 mm to (75.6, 103.9), turned to 0 degrees
- moved D2 47.6 mm to (75.5, 113.7), turned to 180 degrees
- moved BT1 44.8 mm to (75.6, 103.9), turned to 180 degrees
- moved Y1 42.6 mm to (82.2, 99.1), turned to 90 degrees
- moved L2 40.8 mm to (76.2, 110.0), turned to 90 degrees
- moved J1 40.7 mm to (72.6, 94.2), turned to 75 degrees
- moved U4 40.5 mm to (75.6, 103.9)
- moved U3 40.4 mm to (73.9, 110.3)
- moved C10 40.1 mm to (72.0, 111.1)
- moved C9 39.0 mm to (77.9, 110.2), turned to -90 degrees
- moved R10 38.9 mm to (68.0, 111.8), turned to 90 degrees
- moved R1 38.2 mm to (71.6, 105.3)
- moved R4 38.1 mm to (82.8, 106.6), turned to 0 degrees
- moved C1 38.0 mm to (67.3, 109.6)
- moved C8 37.8 mm to (70.8, 111.8), turned to -90 degrees
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Connections:
- net /CLK2 renamed /CLK3
- R3 pad 1: /CLK2_T -> /CLK3_T
- U2 pad 12: unconnected-(U2-CLK3-Pad12) -> /CLK3_T
- U2 pad 13: /CLK2_T -> unconnected-(U2-CLK2-Pad13)
Routing:
- net GND: track 0.00 -> 87.3 mm, vias 0 -> 7
- net +3V3: track 13.5 -> 68.9 mm
- net Net-(BT1-+): track 3.56 -> 37.6 mm, vias 0 -> 2
- net /MCU_DAC0: track 13.0 -> 32.9 mm, vias 2 -> 4
- net /MCU_SDA: track 11.1 -> 29.4 mm, vias 0 -> 3
- net /MCU_SCL: track 6.07 -> 23.3 mm, vias 0 -> 2
- net Net-(D1-A): track 0.00 -> 13.1 mm
- net /MCU_UPDI: track 0.00 -> 10.1 mm
- net /~{TX_EN}: track 10.9 -> 18.4 mm
- net Net-(Q1-G): track 0.00 -> 7.31 mm
- net Net-(C7-Pad1): track 0.00 -> 5.78 mm
- net Net-(U2-XA): track 7.35 -> 1.82 mm
- net /CLK3: track 0.00 -> 5.46 mm
- net Net-(U2-XB): track 9.97 -> 6.16 mm
- net Net-(BZ1-+): track 0.00 -> 3.47 mm
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- added copper zone on B.Cu, net GND
- added copper zone on F.Cu, net GND
Other:
- board size 40 x 40 mm -> 24.4 x 24.4 mm
