File: Transmitter/KiCAD/Button Transmitter/Si5351B-ATtiny412 Dev Board/CR2032 Battery/button_transmitter.kicad_sch (KiCad schematic)
At the start: 37 parts, among them J1 1.27mm Pogo Pads, J2 Conn_Coaxial, Q1 MMUN2238LT1G, U1 ATtiny412-SS, U2 Si5351B-B-GM1, U3 TLV62568DRL, Y1 25MHz

Commit message: Pause point in CR2032 layout
Parts:
- BT1: value JST Battery Connector -> CR2032; footprint Library:JST_PH_HORIZONTAL_WITH_BATTERY_3 -> Battery:BatteryHolder_Keystone_3034_1x20mm
- J2: footprint Library:MountingHole_4.3mm_Pad_Coaxial_2 -> Library:RF_Solder_Pad
- U4: footprint Library:Case -> Library:Case_CR2032
Connections:
- net CLK3_T: now reaches U2.12 (CLK3)
- net CLK3_T: now also R3.1
- net CLK2 renamed CLK3
- net CLK2_T: no longer names the net of U2.13 (CLK2)
- net CLK2_T: no longer R3.1
Other:
- moved on the sheet: J2, R3
Changed lines of the file:
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@@
 	)
 	(no_connect
-		(at 177.165 48.26)
+		(at 177.165 43.18)
 	)
 	(no_connect
-		(at 177.165 43.18)
+		(at 177.165 48.26)
 	)
 	(no_connect
-		(at 177.165 58.42)
+		(at 177.165 53.34)
 	)
 	(wire
@@
 	(wire
 		(pts
-			(xy 194.31 53.34) (xy 205.105 53.34)
+			(xy 194.31 58.42) (xy 205.105 58.42)
 		)
 		(stroke
@@
 	(wire
 		(pts
-			(xy 177.165 53.34) (xy 186.69 53.34)
+			(xy 177.165 58.42) (xy 186.69 58.42)
 		)
 		(stroke
@@
 		)
 	)
-	(label "CLK2_T"
-		(at 177.8 53.34 0)
+	(label "CLK3_T"
+		(at 177.8 58.42 0)
 		(fields_autoplaced yes)
 		(effects
@@
 		)
 	)
-	(label "CLK2"
-		(at 196.215 53.34 0)
+	(label "CLK3"
+		(at 196.215 58.42 0)
 		(fields_autoplaced yes)
 		(effects
@@
 	(symbol
 		(lib_id "power:GND")
-		(at 210.185 58.42 0)
+		(at 210.185 63.5 0)
 		(mirror y)
 		(unit 1)
@@
 		(fields_autoplaced yes)
 		(property "Reference" "#PWR011"
-			(at 210.185 64.77 0)
+			(at 210.185 69.85 0)
 			(effects
 				(font
@@
 		)
 		(property "Value" "GND"
-			(at 210.185 61.5949 90)
+			(at 210.185 66.6749 90)
 			(effects
 				(font
@@
 		)
 		(property "Footprint" ""
-			(at 210.185 58.42 0)
+			(at 210.185 63.5 0)
 			(effects
 				(font
@@
 		)
 		(property "Datasheet" ""
-			(at 210.185 58.42 0)
+			(at 210.185 63.5 0)
 			(effects
 				(font
@@
 		)
 		(property "Description" ""
-			(at 210.185 58.42 0)
+			(at 210.185 63.5 0)
 			(effects
 				(font
@@
 			)
 		)
-		(property "Footprint" "Library:Case"
+		(property "Footprint" "Library:Case_CR2032"
 			(at 243.205 102.87 0)
 			(effects
@@
 	(symbol
 		(lib_id "Connector:Conn_Coaxial")
-		(at 210.185 53.34 0)
+		(at 210.185 58.42 0)
 		(unit 1)
 		(exclude_from_sim no)
@@
 		(fields_autoplaced yes)
 		(property "Reference" "J2"
-			(at 212.7251 52.4211 0)
+			(at 212.7251 57.5011 0)
 			(effects
 				(font
@@
 		)
 		(property "Value" "Conn_Coaxial"
-			(at 212.7251 54.8453 0)
+			(at 212.7251 59.9253 0)
 			(effects
 				(font
@@
 			)
 		)
-		(property "Footprint" "Library:MountingHole_4.3mm_Pad_Coaxial_2"
-			(at 210.185 53.34 0)
+		(property "Footprint" "Library:RF_Solder_Pad"
+			(at 210.185 58.42 0)
 			(effects
 				(font
@@
 			)
 		)
-		(property "Datasheet" " ~"
-			(at 210.185 53.34 0)
+		(property "Datasheet" "~"
+			(at 210.185 58.42 0)
 			(effects
 				(font
@@
 		)
 		(property "Description" ""
-			(at 210.185 53.34 0)
+			(at 210.185 58.42 0)
 			(effects
 				(font
@@
 			)
 		)
-		(property "Value" "JST Battery Connector"
+		(property "Value" "CR2032"
 			(at 73.914 150.5006 0)
 			(effects
@@
 			)
 		)
-		(property "Footprint" "Library:JST_PH_HORIZONTAL_WITH_BATTERY_3"
+		(property "Footprint" "Battery:BatteryHolder_Keystone_3034_1x20mm"
 			(at 76.835 149.606 90)
 			(effects
@@
 	(symbol
 		(lib_id "Device:R_US")
-		(at 190.5 53.34 90)
+		(at 190.5 58.42 90)
 		(unit 1)
 		(exclude_from_sim no)
@@
 		(dnp no)
 		(property "Reference" "R3"
-			(at 187.96 50.8 90)
+			(at 187.96 55.88 90)
 			(effects
 				(font
@@
 		)
 		(property "Value" "0R"
-			(at 193.04 50.8 90)
+			(at 193.04 55.88 90)
 			(effects
 				(font
@@
 		)
 		(property "Footprint" "Resistor_SMD:R_0402_1005Metric"
-			(at 190.754 52.324 90)
+			(at 190.754 57.404 90)
 			(effects
 				(font
@@
 		)
 		(property "Datasheet" "~"
-			(at 190.5 53.34 0)
+			(at 190.5 58.42 0)
 			(effects
 				(font
@@
 		)
 		(property "Description" ""
-			(at 190.5 53.34 0)
+			(at 190.5 58.42 0)
 			(effects
 				(font
