File: Transmitter/KiCAD/Button Transmitter/Si5351B-ATtiny412 Dev Board/CR2032 Battery Buck/button_transmitter.kicad_sch (KiCad schematic)
At the start: 37 parts, among them J1 1.27mm Pogo Pads, J2 Conn_Coaxial, Q1 MMUN2238LT1G, U1 ATtiny412-SS, U2 Si5351B-B-GM1, U3 TLV62568DRL, Y1 25MHz

Commit message: Finished CR2032 layout
I realize now that I should replace the buck converter with a boost converter, going to make a modified version that uses that instead
Parts:
- C10: value 4.7uF -> 10uF
- D2: value CM1213A-01SO -> LS0504EVT233
- R7: value 5M -> 1M
Changed lines of the file:
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@@
 		(fields_autoplaced yes)
 		(property "Reference" "C10"
-			(at 110.8964 147.5811 0)
-			(effects
-				(font
-					(size 1.27 1.27)
-				)
-				(justify left)
-			)
-		)
-		(property "Value" "4.7uF"
+			(at 110.8964 147.581 0)
+			(effects
+				(font
+					(size 1.27 1.27)
+				)
+				(justify left)
+			)
+		)
+		(property "Value" "10uF"
 			(at 110.8964 150.0053 0)
 			(effects
@@
 			)
 		)
-		(property "Value" "5M"
+		(property "Value" "1M"
 			(at 84.709 99.6371 0)
 			(effects
@@
 			)
 		)
-		(property "Value" "CM1213A-01SO"
+		(property "Value" "LS0504EVT233"
 			(at 93.6625 141.7899 0)
 			(effects
@@
 			)
 		)
-		(property "Datasheet" "http://www.onsemi.com/pub_link/Collateral/CM1213A-D.PDF"
+		(property "Datasheet" "https://mm.digikey.com/Volume0/opasdata/d220001/medias/docus/2615/LS0504EVT233_Preliminary_2022.pdf"
 			(at 80.01 142.875 90)
 			(effects
@@
 			)
 		)
-		(property "Description" ""
+		(property "Description" "5V, 4A eFuse with Over Voltage and Over Current Protection"
 			(at 93.98 145.415 0)
 			(effects
