File: Transmitter/KiCAD/Button Transmitter/Si5351B-ATtiny412 Dev Board/CR2032 Battery Boost/button_transmitter.kicad_pcb (KiCad board)
At the start: 2 copper layers, 25 x 25 mm, 40 parts, among them J1 Antenna Screw Pad, J2 1.27mm Pogo Pads For Programm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, Q1 MMUN2238LT1G, U1 TPS22919DCK, U2 Si5351B-B-GM1, U3 ATtiny416-M, U4 Case, U5 TLV61070ADBV, Y1 25MHz

Commit message: Remade gerber files, sent to JLCPCB
Other:
- board text added: "Jan. 2025"
- board text added: "Rev. A"
