File: Transmitter/KiCAD/Button Transmitter/Prototypes/Si5351B-ATtiny416 Dev B/button_transmitter_revb.kicad_sch (KiCad schematic)
At the start: 40 parts, among them J1 Antenna Spring, J2 1.27mm Pogo Pads For Programm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, Q1 DMN601TK-7, U1 TPS22919DCK, U2 Si5351B-B-GM1, U3 ATtiny416-M, U4 Case, U5 TLV61070ADBV, Y1 25MHz

Commit message: Schematic edits, supercap?
Parts:
- removed C102, C9: 100uF, Capacitor_SMD:C_1206_3216Metric, symbol Device:C_Polarized_Small_US
- removed D2: ESD156B1W, Diode_SMD:D_0201_0603Metric, symbol Device:D_TVS
- added R101: 2k2, Library:Worthington_R_0402_1005Metric, symbol Device:R_Small_US
- C101: value 100uF -> 5F; DigiKey https://www.digikey.com/en/products/detail/vishay-sprague/T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 -> https://www.digikey.com/en/products/detail/ymin/SLX3R8L5050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; DigiKey Part TMCMA0G107MTRF -> SLX3R8L5050511
Connections:
- net +BATT: now also R101.2; no longer BT1.1 (+)
- new net: BT1.1 (+), R101.1

Commit message: Rev B design work
Parts:
- removed C103, C104: 100uF, Capacitor_SMD:C_1206_3216Metric, symbol Device:C_Polarized_Small_US
- removed L2: 4.7uH, Inductor_SMD:L_0805_2012Metric, symbol Device:L_Small
- removed R10: 18k, Library:Worthington_R_0402_1005Metric, symbol Device:R_Small_US
- removed R9: 100k, Library:Worthington_R_0402_1005Metric, symbol Device:R_Small_US
- removed U1: TPS22919DCK, Package_TO_SOT_SMD:SOT-363_SC-70-6, symbol library:TPS22919DCK
- removed U5: TLV61070ADBV, Package_TO_SOT_SMD:SOT-23-6, symbol Regulator_Switching:TLV61070ADBV
- added C102: 1uF, Library:Worthington_C_0402_1005Metric, symbol Device:C_Small
- added D102: D_Schottky, symbol Device:D_Schottky
- added L101: 10uH, symbol Device:L
- added R102: 2k2, Library:Worthington_R_0402_1005Metric, symbol Device:R_Small_US
- added U101: TPP361081, Package_TO_SOT_SMD:TSOT-23-6, symbol library:TPP361081
- added U102: MIC2288YML, Package_DFN_QFN:WDFN-8-1EP_2x2mm_P0.5mm_EP0.8x1.2mm, symbol library:MIC2288YML
- C101: value 5F -> 47uF; DigiKey https://www.digikey.com/en/products/detail/ymin/SLX3R8L5050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 -> https://datasheets.kyocera-avx.com/TAJ.pdf; DigiKey Part SLX3R8L5050511 -> TAJD476K025RNJ; Voltage (none) -> 25V
- D101, D3, R11, R8: now not fitted
- R2, R3: value 4k7 -> 15k
Connections:
- net +3V3_SW is gone; now on net +2V5: C1.1, C106.1, C2.1, R2.2, R3.2, U2.16 (VDD), U2.9 (VDDOA)
- net +2V5: now also L1.2; no longer C105.1, C4.1, U3.4 (VCC)
- net +BATT: now also C105.1, C4.1, U3.4 (VCC); no longer C101.1, L1.2, R101.2
- net GND: now also C102.1, U102.4 (AGND), U102.8 (PGND), U102.EP (PAD); no longer C101.2
- net 2V5_RAIL_EN: now reaches U3.5 (PA4)
- net 2V5_RAIL_EN: now also U101.5 (EN)
- net PWR_EN_5351 renamed BOOST_EN
- net BOOST_EN: now also U102.3 (EN)
- new net: C102.2, L101.1, R101.2, U102.2 (VIN)
- new net: D102.2 (A), L101.2, U102.7 (SW)
- no-connect marks 16 -> 15
Other:
- added sheet Math (Math.kicad_sch)
- note added: "Also considering a version using SLX3R8L5050511 5F super capacitor"
- note removed: "R1 = (V_OUT/V_REF - 1) * R2"
- note removed: "V_REF = 500mV"
- moved on the sheet: BT1, C1, C106, C2, C7, J1, R101, R2, R3, R4, U2, Y1

Commit message: Dev 2 Schematic work
Parts:
- removed C6: 1uF, Library:Worthington_C_0402_1005Metric, symbol Device:C_Small
- added C106: 22uF, Library:Worthington_C_0603_1005Metric, symbol Device:C_Small
- added C108: 1uF, Library:Worthington_C_0402_1005Metric, symbol Device:C_Small
- added C111, C112, C113, C114: 100nF, Library:Worthington_C_0402_1005Metric, symbol Device:C_Small
- added C115: 220pF, Library:Worthington_C_0402_1005Metric, symbol Device:C_Small
- added L103: 4u7H, Library:Worthington_L_0603, symbol Device:L
- added R109: 3M, Library:Worthington_R_0402_1005Metric, symbol Device:R_Small_US
- added R111: 402k, Library:Worthington_R_0402_1005Metric, symbol Device:R_Small_US
- added R112, R113: 1k, Library:Worthington_R_0402_1005Metric, symbol Device:R_Small_US
- added R114: 200k, Library:Worthington_R_0402_1005Metric, symbol Device:R_Small_US
- added R115: 107k, Library:Worthington_R_0402_1005Metric, symbol Device:R_Small_US
- added R116: 127k, Library:Worthington_R_0402_1005Metric, symbol Device:R_Small_US
- added R119: 1k, Library:Worthington_R_0402_1005Metric, symbol Device:R_US
- C101: renamed from C106; value 22uF -> 10uF
- C105: Voltage (none) -> 10V
- C110: renamed from C101; footprint Capacitor_SMD:C_1206_3216Metric -> Library:Worthington_CTant_2917; DigiKey Part TAJD476K025RNJ -> T495X476M035ATE300; Voltage 25V -> 35V
- R104: renamed from R1; value 10k -> 1M
- R117: renamed from R102; value 2k2 -> 5k
- Y101: renamed from Y1; DigiKey (none) -> CX3225SB27000D0FLJCC; Digikey Link (none) -> https://www.digikey.com/en/products/detail/kyocera-avx/CX32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; Field4 CX3225SB25000D0FLJCC -> (none)
- renumbered BT1 to BT101, BZ1 to BZ101, BZ2-1 to BZ2-101, C2 to C102, C1 to C103, C4 to C104, C7 to C107, C102 to C109, D3 to D103, J2 to J101, J1 to J102, L1 to L101, L101 to L102, Q1 to Q101, R2 to R101, R3 to R102, R4 to R103, R5 to R105, R6 to R106, R7 to R107, R8 to R108, R101 to R110, R11 to R118, U2 to U101, U3 to U102, U4 to U103, U102 to U104, U101 to U105
Connections:
- net +2V5: now also C113.2, L103.2, R111.2
- net +BATT: now also C106.1
- net GND: now also C110.2, R117.1, U105.1 (GND), C106.2, C111.1, C113.1, C114.1, C115.1, R114.1, R116.1
- net MCU_DAC0: now also R119.1; no longer C107.2, U101.3 (VC)
- net at L101.1, R105.2: now also C108.1
- net at BZ101.1 (+), R104.1: now also C108.2
- net at R117.2: now also U104.6 (FB), R115.1
- net at U104.1 (OVP): now also C110.1, D102.1 (K), U105.3 (VIN), C111.2, R109.2, R115.2
- net at C109.2, L102.1, U104.2 (VIN): now also R110.1; no longer R110.2
- net at BT101.1 (+): now also R110.2; no longer R110.1
- net CHARGE_AIN7: now reaches U102.8 (PA7)
- net CHARGE_AIN7: now also R113.1
- net at U105.2 (SW): now also C112.2, L103.1
- net at U105.4 (VFB): now also C115.2, R112.2
- net at U105.6 (VBST): now also C112.1
- new net: C114.2, R109.1, R113.2, R114.2
- new net: R111.1, R112.1, R116.2
- new net: C107.2, R119.2, U101.3 (VC)
Other:
- note added: "1.59 kHz Low-Pass Helps smooth DAC Out From ATtiny"
- note added: "1.5mA limited, 200mAh capacity"
- note added: "100mH Inductor and 200nF Piezo Tank Circuit Resonate at ~3.56kHz"
- note added: "1mA LED"
- note added: "3.6kHz Resonant 500 Ohm Impedance"
- note added: "Also considering a version using SLX3R8L5050511 5F super capacitor."
- note added: "Boost to +28V, drains to +4.5V"
- note added: "Charge drain resistor"
- note added: "Charge drain resistor Piezo's don't like being charged w/ DC"
- note added: "Current Limit Resistor Might need to tweak if buzzer takes too long to get going loud."
- note added: "DC Block"
- note added: "Energy stored in 2V5 rail gets dumped when transmission stops, so try to keep these as small as possible"
- note added: "Populate if transmitting causes feedback problems"
- note added: "μC ADC Divider IN: 35 to 4 OUT: 2.18 to 0.25 39.1mV per count 4V = 102 26V = 667 35 = 895"
- note removed: "3.6kHz 500 Ohm Impedance"
- note removed: "Also considering a version using SLX3R8L5050511 5F super capacitor"
- moved on the sheet: BT101, BZ101, C101, C102, C103, C104, C107, C109, C110, D101, D102, D103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

Commit message: More Dev B schematic tweaks
Parts:
- renumbered C108 to C107, C107 to C108, D103 to D101, D101 to D102, D102 to D103, R118 to R103, R103 to R104, R119 to R105, R104 to R106, R105 to R107, R106 to R108, R107 to R109, R108 to R110, R109 to R111, R110 to R112, R111 to R113, R112 to R114, R113 to R115, R114 to R116, R115 to R117, R116 to R118, R117 to R119
Connections:
- net BOOST_EN: now also U102.10 (PB4); no longer U102.6 (PA5)
- net MCU_SCL: now also R102.1, U102.1 (PA2); no longer R101.1, U102.14 (PB0)
- net MCU_SDA: now also R101.1, U102.20 (PA1); no longer R102.1, U102.13 (PB1)
Other:
- note added: "UPDI: PA0 SDA: PB1 alt PA1 SCL: PB0 alt PA2 TCA0 WO0: PB0 alt PB3 TCA0 WO1: PB1 alt PB4 TCB0 WO: PA5 alt PC0 TCD0 WOA/WOB/WOC/WOD: PA4, PA5, PC0, PC1"
- moved on the sheet: R101, R102

Commit message: Beginnings of low power boost converter design
Parts:
- added C116: 47uF, Library:Worthington_CTant_2917, symbol Device:C_Polarized_Small_US
- added C117, C118: 100nF, Library:Worthington_C_0402, symbol Device:C_Small
- added R120: 3M48, Library:Worthington_R_0402, symbol Device:R_Small_US
- added R121: 1k, Library:Worthington_R_0402, symbol Device:R_Small_US
- added R122: 197k, Library:Worthington_R_0402, symbol Device:R_Small_US
- added U106: ATtiny416-M, Package_DFN_QFN:VQFN-20-1EP_3x3mm_P0.4mm_EP1.7x1.7mm, symbol MCU_Microchip_ATtiny:ATtiny416-M
- BT101: footprint Library:BatteryHolder_Keystone_3034_1x20mm_CUTOUT -> Battery:BatteryHolder_Keystone_3034_1x20mm
- C101, C105, C106: footprint Library:Worthington_C_0603_1005Metric -> Library:Worthington_C_0603
- C102, C103, C104, C107, C108, C109, C111, C112, C113, C114, C115: footprint Library:Worthington_C_0402_1005Metric -> Library:Worthington_C_0402
- D103: footprint (none) -> Diode_SMD:D_SOD-523
- L102: footprint (none) -> Library:Worthington_L_0603
- R101: footprint Resistor_SMD:R_0402_1005Metric -> Library:Worthington_R_0402
- R102: footprint Resistor_SMD:R_0603_1608Metric -> Library:Worthington_R_0603
- R103, R104, R105, R106, R107, R108, R109, R110, R111, R112, R113, R114, R115, R116, R117, R118, R119: footprint Library:Worthington_R_0402_1005Metric -> Library:Worthington_R_0402
- renumbered BZ2-101 to BZ102
Connections:
- net 2V5_RAIL_EN: now also U106.5 (PA4); no longer U102.5 (PA4)
- net BOOST_EN: now also U106.10 (PB4); no longer U102.10 (PB4)
- net CHARGE_AIN7: now also U106.8 (PA7); no longer U102.8 (PA7)
- net GND: now also U104.9 (PAD), C116.2, C117.1, C118.1, R122.1; no longer U104.EP (PAD)
- net CLK3_T: now reaches U101.12 (CLK3)
- net CLK3_T: now also R104.1
- net CLK0 renamed CLK3
- net CLK0_T: no longer names the net of U101.7 (CLK1)
- net CLK0_T: no longer R104.1
- new net: C118.2, R120.1, R121.2, R122.2
- new net: C116.1, C117.2, R120.2
- new net: U106.21 (GND), U106.3 (GND)
- new net CHARGE_AINP0: R121.1, U102.8 (PA7)
Other:
- added sheet Charge Pump (ChargePump.kicad_sch)
- note added: "Charge drain resistor Piezos don't like being charged w/ DC"
- note added: "μC Comparator Divider Triggers interrupt when voltage >28V. Internal reference set to 1.5V."
- note removed: "Charge drain resistor Piezo's don't like being charged w/ DC"
- company: Engineer: Thomas Francois - KX0STL -> Engineer: Thomas Francois - KXØSTL
- moved on the sheet: BT101, C109, C110, C111, C112, C113, C114, C115, D103, J102, L102, L103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
